File: electronics/rc-light-controller-ws2812-pic12f1840/rc-light-controller-ws2812-12f1840.sch (EAGLE design)
At the start: 7 parts, among them U1 PIC12F1840-E/SN

Commit message: Update schematics and board layout
Parts:
- removed JP3: ICSP, pinhead:PINHD-1X6
- added CLK, DAT, GND, NC, VDD: PTR1TP18R, testpad:PTR1TP18R
- added VPP: PTR1TP18SQ, testpad:PTR1TP18SQ
- C2: value 10..220uF -> 100u 16V; device rcl:CPOL-EUSMCD -> rcl:CPOL-EU153CLV-0605
- D1: value 1N4004 -> ES2D; device diode:1N4004 -> diode:ES2D
- JP1: value LED WS2812 OUT -> LED OUT
- U1: value PIC12F1840-E/SN -> 12F1840
Connections:
- net GND: now also GND.TP; no longer JP3.3
- net N$2: now also VPP.TP; no longer JP3.1
- net N$4: now also DAT.TP; no longer JP3.4
- net UART_RX: now also CLK.TP; no longer JP3.5
- net VDD: now also VDD.TP; no longer JP3.2
Changed lines of the file:
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@@
 </classes>
 <parts>
-<part name="U1" library="PIC12F1840" deviceset="PIC12F1840-E/SN" device=""/>
-<part name="D1" library="diode" deviceset="1N4004" device=""/>
-<part name="JP1" library="pinhead" deviceset="PINHD-1X3" device="" value="LED WS2812 OUT"/>
+<part name="U1" library="PIC12F1840" deviceset="PIC12F1840-E/SN" device="" value="12F1840"/>
+<part name="D1" library="diode" deviceset="ES2D" device=""/>
+<part name="JP1" library="pinhead" deviceset="PINHD-1X3" device="" value="LED OUT"/>
 <part name="JP2" library="pinhead" deviceset="PINHD-1X3" device="" value="UART IN"/>
 <part name="GND1" library="supply1" deviceset="GND" device=""/>
@@
 <part name="GND3" library="supply1" deviceset="GND" device=""/>
 <part name="C1" library="rcl" deviceset="C-EU" device="C0805K" value="100n"/>
-<part name="C2" library="rcl" deviceset="CPOL-EU" device="SMCD" value="10..220uF"/>
-<part name="JP3" library="pinhead" deviceset="PINHD-1X6" device="" value="ICSP"/>
+<part name="C2" library="rcl" deviceset="CPOL-EU" device="153CLV-0605" value="100u 16V"/>
 <part name="GND4" library="supply1" deviceset="GND" device=""/>
+<part name="VPP" library="testpad" deviceset="PTR1" device="TP18SQ"/>
+<part name="VDD" library="testpad" deviceset="PTR1" device="TP18R"/>
+<part name="GND" library="testpad" deviceset="PTR1" device="TP18R"/>
+<part name="DAT" library="testpad" deviceset="PTR1" device="TP18R"/>
+<part name="CLK" library="testpad" deviceset="PTR1" device="TP18R"/>
+<part name="NC" library="testpad" deviceset="PTR1" device="TP18R"/>
 </parts>
 <sheets>
@@
 Replace diode with wire
 when BEC is 5V.</text>
-<text x="88.9" y="-2.54" size="1.778" layer="91">Programming
+<text x="88.9" y="-5.08" size="1.778" layer="91">Programming
 connector</text>
 <text x="-50.8" y="60.96" size="1.778" layer="91">Input from "pre-processor"</text>
@@
 <instances>
 <instance part="U1" gate="A" x="63.5" y="53.34"/>
-<instance part="D1" gate="1" x="10.16" y="83.82"/>
+<instance part="D1" gate="G$1" x="10.16" y="83.82"/>
 <instance part="JP1" gate="A" x="139.7" y="43.18" rot="MR180"/>
 <instance part="JP2" gate="A" x="-20.32" y="50.8" rot="R180"/>
@@
 <attribute name="VALUE" x="12.7" y="43.18" size="1.778" layer="96" rot="R90"/>
 </instance>
-<instance part="JP3" gate="A" x="99.06" y="7.62" rot="MR270"/>
 <instance part="GND4" gate="1" x="78.74" y="10.16"/>
+<instance part="VPP" gate="G$1" x="91.44" y="7.62"/>
+<instance part="VDD" gate="G$1" x="96.52" y="7.62"/>
+<instance part="GND" gate="G$1" x="101.6" y="7.62"/>
+<instance part="DAT" gate="G$1" x="106.68" y="7.62"/>
+<instance part="CLK" gate="G$1" x="111.76" y="7.62"/>
+<instance part="NC" gate="G$1" x="116.84" y="7.62"/>
 </instances>
 <busses>
@@
 <segment>
 <pinref part="C1" gate="G$1" pin="1"/>
-<pinref part="D1" gate="1" pin="C"/>
+<pinref part="D1" gate="G$1" pin="C"/>
 <wire x1="12.7" y1="83.82" x2="22.86" y2="83.82" width="0.1524" layer="91"/>
 <wire x1="22.86" y1="83.82" x2="22.86" y2="55.88" width="0.1524" layer="91"/>
@@
 <pinref part="JP1" gate="A" pin="2"/>
 <wire x1="127" y1="43.18" x2="137.16" y2="43.18" width="0.1524" layer="91"/>
-<pinref part="JP3" gate="A" pin="2"/>
-<wire x1="93.98" y1="25.4" x2="93.98" y2="10.16" width="0.1524" layer="91"/>
+<wire x1="96.52" y1="25.4" x2="96.52" y2="10.16" width="0.1524" layer="91"/>
 <pinref part="U1" gate="A" pin="VDD"/>
 <wire x1="38.1" y1="55.88" x2="33.02" y2="55.88" width="0.1524" layer="91"/>
 <wire x1="33.02" y1="55.88" x2="33.02" y2="25.4" width="0.1524" layer="91"/>
-<wire x1="33.02" y1="25.4" x2="93.98" y2="25.4" width="0.1524" layer="91"/>
+<wire x1="33.02" y1="25.4" x2="96.52" y2="25.4" width="0.1524" layer="91"/>
 <wire x1="33.02" y1="55.88" x2="22.86" y2="55.88" width="0.1524" layer="91"/>
 <junction x="33.02" y="55.88"/>
@@
 <wire x1="22.86" y1="55.88" x2="15.24" y2="55.88" width="0.1524" layer="91"/>
 <wire x1="15.24" y1="55.88" x2="15.24" y2="53.34" width="0.1524" layer="91"/>
+<pinref part="VDD" gate="G$1" pin="TP"/>
 </segment>
 </net>
@@
 </segment>
 <segment>
-<pinref part="JP3" gate="A" pin="3"/>
-<wire x1="96.52" y1="10.16" x2="96.52" y2="20.32" width="0.1524" layer="91"/>
+<wire x1="101.6" y1="10.16" x2="101.6" y2="20.32" width="0.1524" layer="91"/>
 <pinref part="GND4" gate="1" pin="GND"/>
-<wire x1="96.52" y1="20.32" x2="78.74" y2="20.32" width="0.1524" layer="91"/>
+<wire x1="101.6" y1="20.32" x2="78.74" y2="20.32" width="0.1524" layer="91"/>
 <wire x1="78.74" y1="20.32" x2="78.74" y2="12.7" width="0.1524" layer="91"/>
+<pinref part="GND" gate="G$1" pin="TP"/>
 </segment>
 </net>
@@
 <wire x1="-17.78" y1="50.8" x2="-7.62" y2="50.8" width="0.1524" layer="91"/>
 <wire x1="-7.62" y1="50.8" x2="-7.62" y2="83.82" width="0.1524" layer="91"/>
-<pinref part="D1" gate="1" pin="A"/>
+<pinref part="D1" gate="G$1" pin="A"/>
 <wire x1="-7.62" y1="83.82" x2="7.62" y2="83.82" width="0.1524" layer="91"/>
 </segment>
@@
 <pinref part="U1" gate="A" pin="RA1/ICSPCLK"/>
 <wire x1="101.6" y1="53.34" x2="88.9" y2="53.34" width="0.1524" layer="91"/>
-<pinref part="JP3" gate="A" pin="5"/>
-<wire x1="101.6" y1="10.16" x2="101.6" y2="53.34" width="0.1524" layer="91"/>
+<wire x1="111.76" y1="10.16" x2="111.76" y2="53.34" width="0.1524" layer="91"/>
+<wire x1="111.76" y1="53.34" x2="101.6" y2="53.34" width="0.1524" layer="91"/>
 <junction x="101.6" y="53.34"/>
 <label x="0" y="71.12" size="1.778" layer="95"/>
+<pinref part="CLK" gate="G$1" pin="TP"/>
 </segment>
 </net>
@@
 <wire x1="38.1" y1="48.26" x2="35.56" y2="48.26" width="0.1524" layer="91"/>
 <wire x1="35.56" y1="48.26" x2="35.56" y2="27.94" width="0.1524" layer="91"/>
-<pinref part="JP3" gate="A" pin="1"/>
 <wire x1="35.56" y1="27.94" x2="91.44" y2="27.94" width="0.1524" layer="91"/>
 <wire x1="91.44" y1="27.94" x2="91.44" y2="10.16" width="0.1524" layer="91"/>
+<pinref part="VPP" gate="G$1" pin="TP"/>
 </segment>
 </net>
 <net name="N$4" class="0">
 <segment>
-<pinref part="JP3" gate="A" pin="4"/>
-<wire x1="99.06" y1="10.16" x2="99.06" y2="55.88" width="0.1524" layer="91"/>
+<wire x1="106.68" y1="10.16" x2="106.68" y2="55.88" width="0.1524" layer="91"/>
 <pinref part="U1" gate="A" pin="RA0/ICSPDAT"/>
-<wire x1="99.06" y1="55.88" x2="88.9" y2="55.88" width="0.1524" layer="91"/>
+<wire x1="106.68" y1="55.88" x2="88.9" y2="55.88" width="0.1524" layer="91"/>
+<pinref part="DAT" gate="G$1" pin="TP"/>
 </segment>
 </net>

Commit message: Improve the board layout
Parts:
- removed JP2: UART IN, pinhead:PINHD-1X3
- added JP6, JP7: (no value), pinhead:PINHD-2X3
- CLK, DAT, GND, NC, VDD: value PTR1TP18R -> PTR1TP14R; device testpad:PTR1TP18R -> testpad:PTR1TP14R
- VPP: value PTR1TP18SQ -> PTR1TP14SQ; device testpad:PTR1TP18SQ -> testpad:PTR1TP14SQ
Connections:
- removed net N$2: U1.!MCLR!/VPP/RA3, VPP.TP
- removed net N$4: DAT.TP, U1.RA0/ICSPDAT
- removed net UART_RX: CLK.TP, JP2.3, U1.RA1/ICSPCLK
- new net CH3: JP7.5, U1.!MCLR!/VPP/RA3, VPP.TP
- new net OUT/TX: DAT.TP, JP7.6, U1.RA0/ICSPDAT
- new net ST/RX: CLK.TP, JP6.5, U1.RA1/ICSPCLK
- new net TH: JP6.6, U1.RA2
- net GND: now also JP6.1, JP6.2, JP7.1, JP7.2; no longer JP2.1
- net VBAT: now also JP6.3, JP6.4, JP7.3, JP7.4; no longer JP2.2
Other:
- note added: "CH3"
- note added: "Out/Tx"
- note added: "ST/Rx"
- note added: "TH"
- note removed: "Input from "pre-processor""
