File: electronics/rc-light-controller/rc-light-controller-tlc5940-lpc812.sch (EAGLE design)
At the start: 35 parts, among them U2 TLC5940PWP

Commit message: Update LPC812 board
Parts:
- removed PAD24: (no value), wirepad:SMD50X100
- added D1: (Diode), diode:ES2D
- added PAD1: CH3, wirepad:SDM80X120
- added PAD27: +5V, wirepad:SDM80X120
- added PAD28: Data out, wirepad:SDM80X120
- added PAD7: GND, wirepad:SDM80X120
- added R6: 1k, rcl:R-EU_R0603
- PAD6: value CH3/ISP -> OUT/ISP
- R2: value 10k-100k -> 33k; device rcl:R-EU_R0805 -> rcl:R-EU_R0603
- R3, R4: device rcl:R-EU_R0805 -> rcl:R-EU_R0603
- R5: value 1k -> 33k; device rcl:R-EU_R0805 -> rcl:R-EU_R0603
- U$2: device LPC800:LPC812M101JDH16 -> LPC810:LPC812M101JDH16
Connections:
- removed net N$19: PAD6.P, R5.1
- new net N$1: PAD1.P, R6.1
- new net N$2: R6.2, U$2.PIO0_13
- new net N$3: D1.C, PAD27.P
- new net N$5: PAD28.P, U$2.PIO0_9/XTALOUT
- net +3V3: now also R5.1
- net GND: now also PAD7.P
- net N$20: now also PAD6.P
- net VIN: now also D1.A; no longer PAD24.P
Other:
- moved on the sheet: PAD6, R5, U$2
