File: tools/test-jig/electronics/test-jig.kicad_pcb (KiCad board)
At the start: 2 copper layers, 100 x 100 mm, 80 parts, among them J1 POWER, J10 PP3CH_GND_PLUS_S, J11 PP3CH_S, J12 PP8CH_ST1, J13 PP8CH_ST2, J14 PP8CH_TH1, J15 PP8CH_TH2, J16 PP8CH_AUX, J17 PP8CH_AUX2, J18 PP8CH_AUX3, J19 PP8CH_Light, J2 USB_B_Micro, J20 TP_PLUS, J21 TP_GND, J22 TP_ST, J23 TP_TH, J24 TP_AUX, J25 TP_AUX2, J26 TP_AUX3, J27 TP_Light, J28 TP_OUT_ISP, J29 UART_PP, J3 RXe_AUX3, J30 UART_LC, J31 LC_PP, J32 LC_SERVO, J33 LED_PLUS, J34 OUT0, J35 OUT1, J36 OUT2, J37 OUT3, J38 OUT4, J39 OUT5, J4 RXe_AUX2, J40 OUT6, J41 OUT7, J42 OUT8, J43 OUT9, J44 OUT10, J45 OUT11, J46 OUT12, J47 OUT13, J48 OUT14, J49 OUT15, J5 RXe_AUX, J50 OUT15S, J6 RXe_TH, J7 RXe_ST, J8 RX8CH_S_PLUS, J9 RX8CH_GND, SW1 On/Off, SW2 SW_AUX

Commit message: Finalize the PCB for the test jig
Parts:
- J28: footprint Connector_PinHeader_2.54mm:PinHeader_1x02_P2.54mm_Vertical -> Connector_PinHeader_2.54mm:PinHeader_1x03_P2.54mm_Vertical
- J33, J34, J35, J36, J37, J38, J39, J40, J41, J42, J43, J44, J45, J46, J47, J48, J49, J50: footprint TestPoint:TestPoint_THTPad_D1.5mm_Drill0.7mm -> Pogo_pin:Pogo_pin_Drill1mm
- J8: footprint Connector_PinSocket_2.54mm:PinSocket_2x08_P2.54mm_Vertical -> Connector_PinSocket_2.54mm:PinSocket_1x03_P2.54mm_Vertical
- J9: value RX8CH_GND -> RX8CH_S; footprint Connector_PinSocket_2.54mm:PinSocket_1x08_P2.54mm_Vertical -> Connector_PinSocket_2.54mm:PinSocket_1x07_P2.54mm_Vertical
- SW1: footprint Button_Switch_THT:SW_CuK_JS202011CQN_DPDT_Straight -> Connector_PinSocket_2.54mm:PinSocket_2x03_P2.54mm_Vertical
- moved J9 5.45 mm to (146.1, 94.0)
- moved J8 2.92 mm to (151.1, 91.4), turned to 270 degrees
- moved J28 2.24 mm to (148.0, 54.0)
- moved SW1 1.92 mm to (105.9, 54.0), turned to 90 degrees
- moved D1 1.62 mm to (118.6, 55.4)
- moved R1 1.62 mm to (118.6, 61.0)
- moved J27 0.46 mm to (191.5, 58.0)
- turned J38 to 90 degrees
- turned J39 to 90 degrees
- turned J40 to 90 degrees
- turned J41 to 90 degrees
- turned J42 to 90 degrees
- turned J43 to 90 degrees
- turned J44 to 90 degrees
- turned J45 to 90 degrees
Connections:
- J28 pad 1: /OUT_ISP -> GND
- J28 pad 2: /OUT_ISP -> VCC
- J8 pad 1: VCC -> GND
- J8 pad 2: /ST -> VCC
- J8 pad 3: VCC -> /ST
- J9 pad 1: GND -> /TH
- J9 pad 2: GND -> /AUX
- J9 pad 3: GND -> /AUX2
- J9 pad 4: GND -> /AUX3
- J9 pad 5: GND -> (no net)
- J9 pad 6: GND -> (no net)
- J9 pad 7: GND -> (no net)
Routing:
- net GND: track 7.50 -> 0.00 mm
- net /AUX: track 103.4 -> 109.4 mm, vias 2 -> 0
- net /TH: track 111.0 -> 115.1 mm, vias 2 -> 0
- net VCC: track 205.5 -> 209.6 mm
- net Net-(J1-Pad2): track 35.1 -> 31.4 mm
- net Net-(J31-Pad5): track 22.0 -> 25.0 mm
- net /OUT_ISP: track 30.0 -> 27.2 mm
- net /AUX3: track 66.0 -> 68.7 mm, vias 2 -> 0
- net /AUX2: track 65.5 -> 67.0 mm, vias 2 -> 0
Other:
- board text added: "-"
- board text added: "LANE Boys RC Light Controller Mk4 test jig"
- board text added: "OUT"
- board text added: "Pre-Processor 5CH"
- board text added: "ST/Rx"
- board text added: "TH/Tx"
- board text added: "Vcc"
- board text removed: "Pre-Processor 8CH"
