File: tools/test-jig/electronics/test-jig.sch (KiCad schematic (older format))
At the start: 80 parts, among them J1 POWER, J10 PP3CH_GND_PLUS_S, J11 PP3CH_S, J12 PP8CH_ST1, J13 PP8CH_ST2, J14 PP8CH_TH1, J15 PP8CH_TH2, J16 PP8CH_AUX, J17 PP8CH_AUX2, J18 PP8CH_AUX3, J19 PP8CH_Light, J2 USB_B_Micro, J20 TP_PLUS, J21 TP_GND, J22 TP_ST, J23 TP_TH, J24 TP_AUX, J25 TP_AUX2, J26 TP_AUX3, J27 TP_Light, J28 TP_OUT_ISP, J29 UART_PP, J3 RXe_AUX3, J30 UART_LC, J31 LC_PP, J32 LC_SERVO, J33 LED_PLUS, J34 OUT0, J35 OUT1, J36 OUT2, J37 OUT3, J38 OUT4, J39 OUT5, J4 RXe_AUX2, J40 OUT6, J41 OUT7, J42 OUT8, J43 OUT9, J44 OUT10, J45 OUT11, J46 OUT12, J47 OUT13, J48 OUT14, J49 OUT15, J5 RXe_AUX, J50 OUT15S, J6 RXe_TH, J7 RXe_ST, J8 RX8CH_S_PLUS, J9 RX8CH_GND, SW1 On/Off, SW2 SW_AUX

Commit message: Finalize the PCB for the test jig
Parts:
- removed J28: TP_OUT_ISP, Connector_PinHeader_2.54mm:PinHeader_1x02_P2.54mm_Vertical, symbol Connector_Generic:Conn_01x02
- added J28: TP_OUT_ISP, Connector_PinHeader_2.54mm:PinHeader_1x03_P2.54mm_Vertical, symbol Connector_Generic:Conn_01x03
- J33, J34, J35, J36, J37, J38, J39, J40, J41, J42, J43, J44, J45, J46, J47, J48, J49, J50: footprint TestPoint:TestPoint_THTPad_D1.5mm_Drill0.7mm -> Pogo_pin:Pogo_pin_Drill1mm
- J8: footprint Connector_PinSocket_2.54mm:PinSocket_2x08_P2.54mm_Vertical -> Connector_PinSocket_2.54mm:PinSocket_1x03_P2.54mm_Vertical; symbol Connector_Generic:Conn_02x08_Odd_Even -> Connector_Generic:Conn_01x03
- J9: value RX8CH_GND -> RX8CH_S; footprint Connector_PinSocket_2.54mm:PinSocket_1x08_P2.54mm_Vertical -> Connector_PinSocket_2.54mm:PinSocket_1x07_P2.54mm_Vertical; symbol Connector_Generic:Conn_01x08 -> Connector_Generic:Conn_01x07
- SW1: footprint Button_Switch_THT:SW_CuK_JS202011CQN_DPDT_Straight -> Connector_PinSocket_2.54mm:PinSocket_2x03_P2.54mm_Vertical
Connections:
- net AUX: now also J9.2 (Pin_2); no longer J8.6 (Pin_6)
- net AUX2: now also J9.3 (Pin_3); no longer J8.8 (Pin_8)
- net AUX3: now also J9.4 (Pin_4); no longer J8.10 (Pin_10)
- net GND: now also J8.1 (Pin_1), J28.1 (Pin_1); no longer J9.1 (Pin_1), J9.2 (Pin_2), J9.3 (Pin_3), J9.4 (Pin_4), J9.5 (Pin_5), J9.6 (Pin_6), J9.7 (Pin_7), J9.8 (Pin_8)
- net OUT_ISP: now also J28.3 (Pin_3)
- net ST: now also J8.3 (Pin_3); no longer J8.2 (Pin_2)
- net TH: now also J9.1 (Pin_1); no longer J8.4 (Pin_4)
- net VCC: now also J8.2 (Pin_2), J28.2 (Pin_2); no longer J8.1 (Pin_1), J8.11 (Pin_11), J8.13 (Pin_13), J8.15 (Pin_15), J8.3 (Pin_3), J8.5 (Pin_5), J8.7 (Pin_7), J8.9 (Pin_9)
Other:
- note added: "Slave/Servo\noutput"
