File: mk4-tlc5940-lpc812/electronics/rc-light-controller-tlc5940-lpc812.kicad_pcb (KiCad board)
At the start: 2 copper layers, 27 x 18 mm, 42 parts, among them T1 NMOSSOT23, U2 TLC5940PWP

Commit message: Add JLCPCB production number marker
Other:
- board text added: "JLCJLCJLCJLC"
