File: mk4p-tlc5940-lpc812/electronics/rc-light-controller-pinheader-lpc812.sch (KiCad schematic (older format))
At the start: 14 parts, among them J1 Conn_02x17_Odd_Even, J2 Conn_01x06, J3 Conn_01x06, T9 NMOSSOT23, U1 LPC812M101JDH20

Commit message: Change resistor array from concave to convex type.
Convex types seem to be more common, at least on LCSC
Parts:
- RN1: footprint Resistor_SMD:R_Array_Concave_4x0603 -> Resistor_SMD:R_Array_Convex_4x0603
Changed lines of the file:
@@
 F 0 "RN1" V 2033 4300 50  0000 C CNN
 F 1 "R_Pack04" V 2124 4300 50  0000 C CNN
-F 2 "Resistor_SMD:R_Array_Concave_4x0603" V 2725 4300 50  0001 C CNN
+F 2 "Resistor_SMD:R_Array_Convex_4x0603" V 2725 4300 50  0001 C CNN
 F 3 "~" H 2450 4300 50  0001 C CNN
 	1    2450 4300

Commit message: Remove outdated library symbols and footprint
Move everything to KiCAD symbols and footprints, except
for the TLC5940 where we have a custom footprint to
manage the solder paste.
Parts:
- removed 1: TLC5940PWP-rc-light-controller-tlc5940-lpc812-eag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, rc-light-controller-tlc5940-lpc812:SOP65P640X120-29N, symbol rc-light-controller-pinheader-lpc812-rescue:TLC5940PWP-rc-light-controller-tlc5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
- removed U$1: 3V3, rc-light-controller-tlc5940-lpc812:SOT95P300X145-3N, symbol rc-light-controller-pinheader-lpc812-rescue:MCP1703T-3302E_CB-rc-light-controll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
- added U2: TLC5940PWP, rc-light-controller-tlc5940-lpc812:SOP65P640X120-29N, symbol Driver_LED:TLC5940PWP
- added U3: MCP1703A-3302_SOT23, Package_TO_SOT_SMD:SOT-23W, symbol Regulator_Linear:MCP1703A-3302_SOT23
- C1: symbol rc-light-controller-pinheader-lpc812-rescue:C-EUC0805-rc-light-controller-tlc5940-lpc812-eagle-import -> Device:C
- R1: value R -> 2k 1%
- RN1: value R_Pack04 -> 1k x4
Connections:
- net BLANK: now also U2.2 (BLANK)
- net GND: now also U2.1 (GND), U2.29 (PAD), U3.1 (GND)
- net GSCLK: now also U2.25 (GSCLK)
- net OUT0: now also U2.7 (OUT0)
- net OUT1: now also U2.8 (OUT1)
- net OUT10: now also U2.17 (OUT10)
- net OUT11: now also U2.18 (OUT11)
- net OUT12: now also U2.19 (OUT12)
- net OUT13: now also U2.20 (OUT13)
- net OUT14: now also U2.21 (OUT14)
- net OUT15: now also U2.22 (OUT15)
- net OUT2: now also U2.9 (OUT2)
- net OUT3: now also U2.10 (OUT3)
- net OUT4: now also U2.11 (OUT4)
- net OUT5: now also U2.12 (OUT5)
- net OUT6: now also U2.13 (OUT6)
- net OUT7: now also U2.14 (OUT7)
- net OUT8: now also U2.15 (OUT8)
- net OUT9: now also U2.16 (OUT9)
- net SCLK: now also U2.4 (SCLK)
- net SIN: now also U2.5 (SIN)
- net VIN: now also U3.3 (VI)
- net XLAT: now also U2.3 (XLAT)
- net +3V3: now reaches C2.1
- net +3V3: now also C3.1, U1.15 (VDD), U2.26 (DCPRG), U2.28 (VCC), U2.6 (VPRG), U3.2 (VO)
- net OUT15S_OUT: now reaches J1.2 (Pin_2), T9.3 (D)
- net at R1.1: now also U2.27 (IREF)
- no-connect marks 11 -> 10
Other:
- note added: "LDO: \nMCP1702, MCP1703\nME6209A33M3G"
- note added: "LED driver"
- note added: "LED output"
- note added: "N-Channel MOSFET\nSOT23 package\ne.g. PMV16UN, PMV30UN, \nSI2302. AO3400, DMN2075U-7"
- note added: "Output connector"
- note added: "Servo/Pre-processor in/out"
- note added: "Switched output driver"
- note added: "X7R or X5R"
- note removed: "LDO: Microchip \nMCP1702 or MCP1703"
- note removed: "LED driver and outputs"
- note removed: "N-Channel MOSFET\nSOT23 package\ne.g. NXP PMV16UN"
- note removed: "Servo in/out"
- note removed: "Slave out"
- note removed: "X7R"
- moved on the sheet: C2, C3, H1, H2, J1, J2, J3, R1, RN1, T9, U1

Commit message: Add README and tweak silkscreen and fab layers
Parts:
- T9: value NMOSSOT23 -> PMV30UN
Changed lines of the file:
@@
 U 1 1 5EEE69E5
 P 11150 6800
-F 0 "T9" H 11250 6900 59  0000 L BNN
-F 1 "NMOSSOT23" H 11250 6800 59  0001 L BNN
+F 0 "T9" H 11050 6950 59  0000 L BNN
+F 1 "PMV30UN" H 11250 6800 59  0001 L BNN
 F 2 "Package_TO_SOT_SMD:SOT-23" H 11150 6800 50  0001 C CNN
 F 3 "" H 11150 6800 50  0001 C CNN
@@
 	4700 2300 5250 2300
 $Comp
-L power:+3V3 #PWR?
+L power:+3V3 #PWR05
 U 1 1 5F1AFD5A
 P 5250 1900
-F 0 "#PWR?" H 5250 1750 50  0001 C CNN
+F 0 "#PWR05" H 5250 1750 50  0001 C CNN
 F 1 "+3V3" H 5265 2073 50  0000 C CNN
 F 2 "" H 5250 1900 50  0001 C CNN
@@
 $EndComp
 $Comp
-L power:+3V3 #PWR?
+L power:+3V3 #PWR08
 U 1 1 5F1B1B4B
 P 8700 2100
-F 0 "#PWR?" H 8700 1950 50  0001 C CNN
+F 0 "#PWR08" H 8700 1950 50  0001 C CNN
 F 1 "+3V3" H 8715 2273 50  0000 C CNN
 F 2 "" H 8700 2100 50  0001 C CNN
@@
 $EndComp
 $Comp
-L power:+3V3 #PWR?
+L power:+3V3 #PWR07
 U 1 1 5F1BA1EF
 P 7700 6650
-F 0 "#PWR?" H 7700 6500 50  0001 C CNN
+F 0 "#PWR07" H 7700 6500 50  0001 C CNN
 F 1 "+3V3" H 7715 6823 50  0000 C CNN
 F 2 "" H 7700 6650 50  0001 C CNN

Commit message: Add datasheets and fix part values
Parts:
- J1: value Conn_02x17_Odd_Even -> Pinheader right-angle 2x17
- J2, J3: value Conn_01x06 -> Pinheader straight 1x06
Changed lines of the file:
@@
 F 1 "47u/6V3" H 5368 2805 50  0000 L CNN
 F 2 "Capacitor_SMD:C_0805_2012Metric" H 5288 2700 50  0001 C CNN
-F 3 "~" H 5250 2850 50  0001 C CNN
+F 3 "https://www.vishay.com/doc?40189" H 5250 2850 50  0001 C CNN
 	1    5250 2850
 	1    0    0    -1
@@
 P 1750 5750
 F 0 "J2" H 1668 5225 50  0000 C CNN
-F 1 "Conn_01x06" H 1668 5316 50  0000 C CNN
+F 1 "Pinheader straight 1x06" H 1668 5316 50  0000 C CNN
 F 2 "rc-light-controller-tlc5940-lpc812:PinHeader_1x06_P2.54mm_Flat" H 1750 5750 50  0001 C CNN
 F 3 "~" H 1750 5750 50  0001 C CNN
@@
 P 1750 7550
 F 0 "J3" H 1668 7025 50  0000 C CNN
-F 1 "Conn_01x06" H 1668 7116 50  0000 C CNN
+F 1 "Pinheader straight 1x06" H 1668 7116 50  0000 C CNN
 F 2 "rc-light-controller-tlc5940-lpc812:PinHeader_1x06_P2.54mm_Flat" H 1750 7550 50  0001 C CNN
 F 3 "~" H 1750 7550 50  0001 C CNN
@@
 P 14000 3350
 F 0 "J1" H 14050 4367 50  0000 C CNN
-F 1 "Conn_02x17_Odd_Even" H 14050 4276 50  0000 C CNN
+F 1 "Pinheader right-angle 2x17" H 14050 4276 50  0000 C CNN
 F 2 "Connector_PinHeader_2.54mm:PinHeader_2x17_P2.54mm_Horizontal" H 14000 3350 50  0001 C CNN
 F 3 "~" H 14000 3350 50  0001 C CNN
@@
 F 1 "PMV30UN" H 11250 6800 59  0001 L BNN
 F 2 "Package_TO_SOT_SMD:SOT-23" H 11150 6800 50  0001 C CNN
-F 3 "" H 11150 6800 50  0001 C CNN
+F 3 "https://assets.nexperia.com/documents/data-sheet/PMV30UN.pdf" H 11150 6800 50  0001 C CNN
 	1    11150 6800
 	1    0    0    -1
@@
 F 1 "1k x4" V 2924 5450 50  0000 C CNN
 F 2 "Resistor_SMD:R_Array_Convex_4x0603" V 3525 5450 50  0001 C CNN
-F 3 "~" H 3250 5450 50  0001 C CNN
+F 3 "https://datasheet.lcsc.com/szlcsc/1810311812_UNI-ROYAL-Uniroyal-Elec-4D03WGJ0102T5E_C20197.pdf" H 3250 5450 50  0001 C CNN
 	1    3250 5450
 	0    1    1    0
