File: mk4-tlc5940-lpc812/electronics-switching-mini5/rc-light-controller-switching-mini5-lpc812.sch (KiCad schematic (older format))
At the start: 20 parts, among them J1 Conn_01x03, J2 Conn_01x03, J3 Pinheader straight 1x06, J4 Conn_01x03, J5 Conn_01x03, J6 Conn_01x03, J7 Conn_01x03, J8 Conn_01x03, J9 Conn_01x03, T1 PMV30UN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

Commit message: Layout Mini5
Connections:
- net GND: now also J3.7 (Pin_7)
- net LED+: now also J3.8 (Pin_8)
- net OUT0: now also T3.1 (G); no longer T1.1 (G)
- net OUT2: now also T1.1 (G); no longer T3.1 (G)
- net ST-RX: now also RN1.4 (R4.1); no longer RN1.1 (R1.1)
- net ST-Rx-in: now also RN1.5 (R4.2); no longer RN1.8 (R1.2)
- net TH-TX: now also RN1.1 (R1.1); no longer RN1.4 (R4.1)
- net TH-Tx-in: now also RN1.8 (R1.2); no longer RN1.5 (R4.2)
- net VIN: now also J3.9 (Pin_9)
Changed lines of the file:
@@
 	12400 3350 12400 3950
 Connection ~ 12400 3950
-Text Label 11450 3150 0    50   ~ 0
+Text Label 11450 4350 0    50   ~ 0
 OUT0
 Wire Wire Line
@@
 Wire Wire Line
 	11450 4350 11800 4350
-Text Label 11450 4350 0    50   ~ 0
+Text Label 11450 3150 0    50   ~ 0
 OUT2
 NoConn ~ 8750 6700
@@
 	6200 6600 7350 6600
 Wire Wire Line
-	5950 6500 6600 6500
-Wire Wire Line
-	6600 6500 6600 7000
+	5950 6800 6600 6800
 Wire Wire Line
 	6600 7000 7350 7000
@@
 Text Label 4300 7050 2    50   ~ 0
 CH3
+Text Label 4850 6500 0    50   ~ 0
+ST-Rx-in
+Wire Wire Line
+	4850 6500 5550 6500
+Wire Wire Line
+	4850 6800 5550 6800
 Text Label 4850 6800 0    50   ~ 0
-ST-Rx-in
-Wire Wire Line
-	4850 6800 5550 6800
-Wire Wire Line
-	4850 6500 5550 6500
-Text Label 4850 6500 0    50   ~ 0
 TH-Tx-in
 $Comp
@@
 NoConn ~ 5550 6600
 Wire Wire Line
-	6200 6600 6200 6800
-Wire Wire Line
-	6200 6800 5950 6800
+	6200 6600 6200 6500
+Wire Wire Line
+	6200 6500 5950 6500
 NoConn ~ 5950 6600
+Wire Wire Line
+	6600 6800 6600 7000
+$Comp
+L power:GND #PWR?
+U 1 1 5FF80AFD
+P 13150 4700
+F 0 "#PWR?" H 13150 4450 50  0001 C CNN
+F 1 "GND" H 13155 4527 50  0000 C CNN
+F 2 "" H 13150 4700 50  0001 C CNN
+F 3 "" H 13150 4700 50  0001 C CNN
+	1    13150 4700
+	1    0    0    -1
+$EndComp
+Wire Wire Line
+	13450 4250 13150 4250
+Wire Wire Line
+	13150 4250 13150 4700
+Wire Wire Line
+	13300 4050 13300 4350
+Wire Wire Line
+	13300 4350 13450 4350
+Connection ~ 13300 4050
+Wire Wire Line
+	13450 4450 12750 4450
+Text Label 12750 4450 0    50   ~ 0
+VIN
 $EndSCHEMATC

Commit message: Fix AUX2 and improve the layout
Parts:
- J1, J2, J4, J5, J6, J7, J8, J9: footprint Connector_PinHeader_2.54mm:PinHeader_1x03_P2.54mm_Vertical -> rc-light-controller-tlc5940-lpc812:PinHeader_1x03_P2.54mm_Vertical_nosilk
- J3: footprint Connector_PinHeader_2.54mm:PinHeader_1x09_P2.54mm_Vertical -> rc-light-controller-tlc5940-lpc812:PinHeader_1x09_P2.54mm_Vertical_nosilk
Connections:
- net AUX2: now also RN2.2 (R2.1), U1.18 (PIO0_6); no longer RN2.3 (R3.1), U1.14 (PIO0_8)
- net AUX2-in: now also RN2.7 (R2.2); no longer RN2.6 (R3.2)
- net AUX3: now also RN2.1 (R1.1); no longer RN2.2 (R2.1)
- net AUX3-in: now also RN2.8 (R1.2); no longer RN2.7 (R2.2)
- net OUT-ISP: now also RN2.3 (R3.1); no longer RN2.1 (R1.1)
- net OUT-ISP-in: now also RN2.6 (R3.2); no longer RN2.8 (R1.2)
- net TH-TX: now also RN1.3 (R3.1); no longer RN1.1 (R1.1)
- net TH-Tx-in: now also RN1.6 (R3.2); no longer RN1.8 (R1.2)
- net CH3 renamed AUX
- net CH3-in renamed AUX-in
Other:
- note added: "Note: Resistor assignment according\nto what is easiest for the layout"
- note added: "We are using PIO0_6 instead of \nPIO0_8 for AUX2 so that in the \nfuture we could make a \n9-output Mk4S with 5-channel input.\n\nWhen switching hardware is detected \n(PIO0_14 is GND) then the software will\nuse PIO0_6 for AUX2, otherwise PIO0_8"
- moved on the sheet: C3, J1, J2, J3, J4, J5, J6, J7, J8, J9, R1, RN1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

Commit message: Add OUT3 to Mk4S-mini5
Parts:
- added T4: PMV30UN, Package_TO_SOT_SMD:SOT-23, symbol Device:Q_NMOS_GSD
- J3: value Pinheader straight 1x06 -> Pinheader straight 1x08; footprint rc-light-controller-tlc5940-lpc812:PinHeader_1x09_P2.54mm_Vertical_nosilk -> rc-light-controller-tlc5940-lpc812:PinHeader_1x08_P2.54mm_Vertical_nosilk; symbol Connector_Generic:Conn_01x09 -> Connector_Generic:Conn_01x08
Connections:
- net GND: now also T4.2 (S); no longer J3.7 (Pin_7)
- net VIN: now also J3.2 (Pin_2), J3.4 (Pin_4), J3.6 (Pin_6), J3.8 (Pin_8); no longer J3.9 (Pin_9)
- net OUT3: now reaches U1.10 (PIO0_16)
- net OUT3: now also T4.1 (G)
- net at T2.3 (D): now also J3.5 (Pin_5); no longer J3.4 (Pin_4)
- net at T3.3 (D): now also J3.7 (Pin_7); no longer J3.6 (Pin_6)
- net at T1.3 (D): now also J3.3 (Pin_3); no longer J3.2 (Pin_2)
- removed net LED+: J3.1 (Pin_1), J3.3 (Pin_3), J3.5 (Pin_5), J3.8 (Pin_8)
- new net: J3.1 (Pin_1), T4.3 (D)
- no-connect marks 12 -> 11
Other:
- note removed: "VIN1 is physically close to LED+.\nThis allows two modes of operation:\n1) when VIN1 is conntected to LED+\nvia a jumper, then the LEDs are \npowered from the receiver.\n2) A separate power supply can be \nconnected to LED+ (and the nearby GND),\ne.g. for higher voltages"
Changed lines of the file:
@@
 Wire Wire Line
 	8450 7000 8450 7100
-Text Notes 11600 1850 0    85   ~ 0
+Text Notes 11600 1150 0    85   ~ 0
 LED driver and outputs
 Text Label 7150 5900 0    50   ~ 0
@@
 OUT2
 NoConn ~ 7750 6400
-Text Notes 14000 4650 0    59   ~ 0
-VIN1 is physically close to LED+.\nThis allows two modes of operation:\n1) when VIN1 is conntected to LED+\nvia a jumper, then the LEDs are \npowered from the receiver.\n2) A separate power supply can be \nconnected to LED+ (and the nearby GND),\ne.g. for higher voltages
 Text Label 2750 4750 2    50   ~ 0
 ST-Rx-in
 Text Label 2750 4850 2    50   ~ 0
 VIN
-Text Label 13600 2000 0    50   ~ 0
-LED+
 Text Label 9800 6300 2    50   ~ 0
 AUX
@@
 	10300 6400 10300 6600
 $Comp
-L Connector_Generic:Conn_01x09 J3
+L Connector_Generic:Conn_01x08 J3
 U 1 1 5FF85660
-P 13950 3200
-F 0 "J3" H 13868 2675 50  0000 C CNN
-F 1 "Pinheader straight 1x06" H 13950 3650 50  0000 C CNN
-F 2 "rc-light-controller-tlc5940-lpc812:PinHeader_1x09_P2.54mm_Vertical_nosilk" H 13950 3200 50  0001 C CNN
-F 3 "~" H 13950 3200 50  0001 C CNN
-	1    13950 3200
+P 13950 3000
+F 0 "J3" H 13868 2475 50  0000 C CNN
+F 1 "Pinheader straight 1x08" H 14250 2350 50  0000 C CNN
+F 2 "rc-light-controller-tlc5940-lpc812:PinHeader_1x08_P2.54mm_Vertical_nosilk" H 13950 3000 50  0001 C CNN
+F 3 "~" H 13950 3000 50  0001 C CNN
+	1    13950 3000
 	1    0    0    -1
 $EndComp
@@
 NoConn ~ 7750 6000
 NoConn ~ 9150 6500
-NoConn ~ 9150 6600
 NoConn ~ 7750 6600
 NoConn ~ 9150 5900
@@
 Wire Wire Line
 	6750 5900 6750 6300
-$Comp
-L power:GND #PWR0107
-U 1 1 5FF80AFD
-P 13450 3850
-F 0 "#PWR0107" H 13450 3600 50  0001 C CNN
-F 1 "GND" H 13455 3677 50  0000 C CNN
-F 2 "" H 13450 3850 50  0001 C CNN
-F 3 "" H 13450 3850 50  0001 C CNN
-	1    13450 3850
-	1    0    0    -1
-$EndComp
-Wire Wire Line
-	13750 3400 13450 3400
-Wire Wire Line
-	13450 3400 13450 3850
-Wire Wire Line
-	13600 3200 13600 3500
-Wire Wire Line
-	13600 3500 13750 3500
-Connection ~ 13600 3200
-Wire Wire Line
-	13750 3600 13050 3600
-Text Label 13050 3600 0    50   ~ 0
+Text Label 13600 2000 0    50   ~ 0
 VIN
 Wire Wire Line
@@
 Text Notes 3550 8300 0    50   ~ 0
 Note: Resistor assignment according\nto what is easiest for the layout
+$Comp
+L Device:Q_NMOS_GSD T4
+U 1 1 60061D05
+P 12300 1650
+F 0 "T4" H 12150 1800 59  0000 L BNN
+F 1 "PMV30UN" H 12400 1650 59  0001 L BNN
+F 2 "Package_TO_SOT_SMD:SOT-23" H 12300 1650 50  0001 C CNN
+F 3 "https://assets.nexperia.com/documents/data-sheet/PMV30UN.pdf" H 12300 1650 50  0001 C CNN
+	1    12300 1650
+	1    0    0    -1
+$EndComp
+Wire Wire Line
+	11750 1650 12100 1650
+Text Label 11750 1650 0    50   ~ 0
+OUT3
+Wire Wire Line
+	12400 1850 12700 1850
+Wire Wire Line
+	12700 1850 12700 2500
+Connection ~ 12700 2500
+Wire Wire Line
+	13600 3200 13600 3400
+Wire Wire Line
+	13600 3400 13750 3400
+Connection ~ 13600 3200
+Wire Wire Line
+	13750 2700 13450 2700
+Wire Wire Line
+	13450 2700 13450 1450
+Wire Wire Line
+	13450 1450 12400 1450
+Wire Wire Line
+	9800 6600 9150 6600
+Text Label 9800 6600 2    50   ~ 0
+OUT3
 $EndSCHEMATC
