File: mk4-tlc5940-lpc812/electronics-switching-mini5/rc-light-controller-switching-mini5-lpc812.kicad_pcb (KiCad board)
At the start: 2 copper layers, 21 x 24 mm, 21 parts, among them J1 Conn_01x03, J2 Conn_01x03, J3 Pinheader straight 1x08, J4 Conn_01x03, J5 Conn_01x03, J6 Conn_01x03, J7 Conn_01x03, J8 Conn_01x03, J9 Conn_01x03, T1 PMV30UN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

Commit message: Add PCB thickness remark
Other:
- board text added: "Thickness 1mm"
