File: mk4-tlc5940-lpc812/electronics/XSON16-version/rc-light-controller-tlc5940-lpc812.sch (KiCad schematic (older format))
At the start: 34 parts, among them T1 NMOSSOT23, U2 TLC5940PWP

Commit message: Tweak layout and schematics
Parts:
- RN1: value R_Pack04 -> 1K
- renumbered U$1 to U1, U$2 to U2, U2 to U3
Connections:
- net ST-IN: now reaches PAD3.1 (Pin_1), RN1.1 (R1.1)
- net OUT15S: now reaches OUT15S1.1 (Pin_1), T1.3 (D)
- net OUT0: now reaches OUT0.1 (Pin_1), U3.7 (OUT0)
- net AUX-IN: now reaches PAD5.1 (Pin_1), RN1.2 (R2.1)
- net OUT-ISP-OUT: now reaches PAD6.1 (Pin_1), RN1.3 (R3.1)
- net TH-IN: now reaches PAD4.1 (Pin_1), RN1.4 (R4.1)
- net OUT1: now reaches OUT1.1 (Pin_1), U3.8 (OUT1)
- net OUT11: now reaches OUT11.1 (Pin_1), U3.18 (OUT11)
- net IREF: now reaches R1.1, U3.27 (IREF)
- net OUT3: now reaches OUT3.1 (Pin_1), U3.10 (OUT3)
- net OUT4: now reaches OUT4.1 (Pin_1), U3.11 (OUT4)
- net OUT5: now reaches OUT5.1 (Pin_1), U3.12 (OUT5)
- net OUT6: now reaches OUT6.1 (Pin_1), U3.13 (OUT6)
- net OUT7: now reaches OUT7.1 (Pin_1), U3.14 (OUT7)
- net OUT8: now reaches OUT8.1 (Pin_1), U3.15 (OUT8)
- net OUT9: now reaches OUT9.1 (Pin_1), U3.16 (OUT9)
- net OUT10: now reaches OUT10.1 (Pin_1), U3.17 (OUT10)
- net OUT12: now reaches OUT12.1 (Pin_1), U3.19 (OUT12)
- net OUT13: now reaches OUT13.1 (Pin_1), U3.20 (OUT13)
- net OUT14: now reaches OUT14.1 (Pin_1), U3.21 (OUT14)
- net OUT15: now reaches OUT15.1 (Pin_1), U3.22 (OUT15)
- net OUT2: now reaches OUT2.1 (Pin_1), U3.9 (OUT2)
- net CH3 renamed AUX
- net OUT/ISP renamed OUT-ISP
- net ST/RX renamed ST-RX
- net TH/TX renamed TH-TX
Other:
- moved on the sheet: OUT15S1, T1
Changed lines of the file:
@@
 Title "DIY RC Light Controller Mk4 Rev4"
 Date "2019-05-01"
-Rev "2"
+Rev "4"
 Comp "LANE Boys RC"
 Comment1 "laneboysrc@gmail.com"
@@
 	5100 2700 5100 3200
 Wire Wire Line
-	2050 4600 2050 2800
-Wire Wire Line
-	2050 2800 1450 2800
+	1550 4600 1550 2800
+Wire Wire Line
+	1550 2800 1450 2800
 Wire Wire Line
 	12300 3900 12300 4050
 Wire Wire Line
-	14150 9000 14150 9100
+	10800 8400 10800 8500
 Text Label 9500 3500 0    70   ~ 0
 SIN
@@
 	5000 7500 4400 7500
 Text Label 4400 7500 0    70   ~ 0
-TH/TX
-Text Label 4550 4350 2    70   ~ 0
-TH/TX
+TH-TX
+Text Label 5050 4350 2    70   ~ 0
+TH-TX
 Wire Wire Line
 	4000 2650 4000 2400
@@
 	5000 7100 4400 7100
 Text Label 4400 7100 0    70   ~ 0
-ST/RX
-Text Label 4550 4050 2    70   ~ 0
-ST/RX
+ST-RX
+Text Label 5050 4050 2    70   ~ 0
+ST-RX
 Wire Wire Line
 	13000 2100 14200 2100
@@
 	7400 7600 6400 7600
 Text Label 7400 7600 2    70   ~ 0
-OUT/ISP
-Text Label 4550 4250 2    70   ~ 0
-OUT/ISP
-Text Label 4550 4150 2    70   ~ 0
-CH3
+OUT-ISP
+Text Label 5050 4250 2    70   ~ 0
+OUT-ISP
+Text Label 5050 4150 2    70   ~ 0
+AUX
 Wire Wire Line
 	7400 7700 6400 7700
 Text Label 7400 7700 2    70   ~ 0
-CH3
-Wire Wire Line
-	14950 8300 14150 8300
-Wire Wire Line
-	14150 8600 14150 8300
+AUX
+Wire Wire Line
+	11600 7700 10800 7700
+Wire Wire Line
+	10800 8000 10800 7700
 Wire Wire Line
 	6400 7300 7400 7300
@@
 OUT-SWITCHED
 Wire Wire Line
-	13850 8800 12750 8800
-Text Label 12750 8800 0    70   ~ 0
+	10500 8200 9400 8200
+Text Label 9400 8200 0    70   ~ 0
 OUT-SWITCHED
 $Comp
-L Driver_LED:TLC5940PWP U2
+L Driver_LED:TLC5940PWP U3
 U 1 1 840783A6
 P 12300 2800
-F 0 "U2" H 11850 3650 59  0000 L BNN
+F 0 "U3" H 11850 3650 59  0000 L BNN
 F 1 "TLC5940PWP" H 13000 3750 59  0000 R TNN
 F 2 "rc-light-controller-tlc5940-lpc812:SOP65P640X120-29N" H 12300 2800 50  0001 C CNN
 F 3 "" H 12300 2800 50  0001 C CNN
 	1    12300 2800
-	1    0    0    -1
-$EndComp
-$Comp
-L power:+3V3 #+3V01
-U 1 1 910CF6D9
-P 5700 6150
-F 0 "#+3V01" H 5700 6150 50  0001 C CNN
-F 1 "+3V3" V 5600 5950 59  0000 L BNN
-F 2 "" H 5700 6150 50  0001 C CNN
-F 3 "" H 5700 6150 50  0001 C CNN
-	1    5700 6150
-	1    0    0    -1
-$EndComp
-$Comp
-L power:+3V3 #+3V02
-U 1 1 BB2FC3B7
-P 12300 1700
-F 0 "#+3V02" H 12300 1700 50  0001 C CNN
-F 1 "+3V3" V 12200 1500 59  0000 L BNN
-F 2 "" H 12300 1700 50  0001 C CNN
-F 3 "" H 12300 1700 50  0001 C CNN
-	1    12300 1700
 	1    0    0    -1
 $EndComp
@@
 F 3 "" H 10900 3850 50  0001 C CNN
 	1    10900 3850
-	1    0    0    -1
-$EndComp
-$Comp
-L power:+3V3 #+3V03
-U 1 1 8A0CCF2D
-P 6000 2100
-F 0 "#+3V03" H 6000 2100 50  0001 C CNN
-F 1 "+3V3" V 5900 1900 59  0000 L BNN
-F 2 "" H 6000 2100 50  0001 C CNN
-F 3 "" H 6000 2100 50  0001 C CNN
-	1    6000 2100
 	1    0    0    -1
 $EndComp
@@
 $EndComp
 $Comp
-L Regulator_Linear:MCP1703A-3302_SOT23 U$1
+L Regulator_Linear:MCP1703A-3302_SOT23 U1
 U 1 1 09B5DC2D
 P 5100 2400
-F 0 "U$1" H 4900 2550 69  0000 L BNN
+F 0 "U1" H 4900 2550 69  0000 L BNN
 F 1 "3V3" H 5200 2050 69  0000 L BNN
 F 2 "Package_TO_SOT_SMD:SOT-23W" H 5100 2400 50  0001 C CNN
@@
 $EndComp
 $Comp
-L MCU_NXP_LPC:LPC812M101JTB16 U$2
+L MCU_NXP_LPC:LPC812M101JTB16 U2
 U 1 1 563110E3
 P 5700 7400
-F 0 "U$2" H 5150 6800 42  0000 L BNN
+F 0 "U2" H 5150 6850 42  0000 L BNN
 F 1 "LPC812" H 5700 7400 50  0001 C CNN
 F 2 "Package_SON:NXP_XSON-16" H 5700 7400 50  0001 C CNN
@@
 L Connector_Generic:Conn_01x01 OUT15S1
 U 1 1 1D8B1813
-P 15150 8300
-F 0 "OUT15S1" H 15105 8373 59  0000 L BNN
-F 1 "SMD50X100" H 15105 8170 59  0001 L BNN
-F 2 "rc-light-controller-tlc5940-lpc812:SMD50X100" H 15150 8300 50  0001 C CNN
-F 3 "" H 15150 8300 50  0001 C CNN
-	1    15150 8300
+P 11800 7700
+F 0 "OUT15S1" H 11755 7773 59  0000 L BNN
+F 1 "SMD50X100" H 11755 7570 59  0001 L BNN
+F 2 "rc-light-controller-tlc5940-lpc812:SMD50X100" H 11800 7700 50  0001 C CNN
+F 3 "" H 11800 7700 50  0001 C CNN
+	1    11800 7700
 	1    0    0    -1
 $EndComp
@@
 L Device:Q_NMOS_GSD T1
 U 1 1 8692C711
-P 14050 8800
-F 0 "T1" H 14250 8850 59  0000 L BNN
-F 1 "NMOSSOT23" H 14150 8800 59  0001 L BNN
-F 2 "Package_TO_SOT_SMD:SOT-23" H 14050 8800 50  0001 C CNN
-F 3 "" H 14050 8800 50  0001 C CNN
-	1    14050 8800
+P 10700 8200
+F 0 "T1" H 10900 8250 59  0000 L BNN
+F 1 "NMOSSOT23" H 10800 8200 59  0001 L BNN
+F 2 "Package_TO_SOT_SMD:SOT-23" H 10700 8200 50  0001 C CNN
+F 3 "" H 10700 8200 50  0001 C CNN
+	1    10700 8200
 	1    0    0    -1
 $EndComp
@@
 Text Notes 1800 2000 0    85   ~ 0
 Servo in/out
-Text Notes 11200 1500 0    85   ~ 0
+Text Notes 11200 1350 0    85   ~ 0
 LED driver and outputs
 Text Notes 4600 1750 0    85   ~ 0
@@
 Text Notes 2650 2650 0    59   ~ 0
 Input voltage range:\n4 ... 10V
-Text Notes 6300 2600 0    59   ~ 0
+Text Notes 4600 2100 0    59   ~ 0
 LDO: Microchip \nMCP1702 or MCP1703
 Text Notes 4150 6750 0    59   ~ 0
@@
 Text Notes 6800 8400 0    59   ~ 0
 NXP LPC812\nARM Cortex-M0\n16K Flash, 4K RAM\nTSSOP-16
-Text Notes 13300 7900 0    85   ~ 0
+Text Notes 9950 7300 0    85   ~ 0
 Switched output\nfor light bar or similar
-Text Notes 14550 9200 0    56   ~ 0
+Text Notes 11200 8600 0    56   ~ 0
 N-Channel MOSFET\nSOT23 package\ne.g. NXP PMV16UN
 NoConn ~ 5000 7600
@@
 L power:GND #PWR0101
 U 1 1 5CCABD51
-P 2050 4600
-F 0 "#PWR0101" H 2050 4350 50  0001 C CNN
-F 1 "GND" H 2055 4427 50  0000 C CNN
-F 2 "" H 2050 4600 50  0001 C CNN
-F 3 "" H 2050 4600 50  0001 C CNN
-	1    2050 4600
+P 1550 4600
+F 0 "#PWR0101" H 1550 4350 50  0001 C CNN
+F 1 "GND" H 1555 4427 50  0000 C CNN
+F 2 "" H 1550 4600 50  0001 C CNN
+F 3 "" H 1550 4600 50  0001 C CNN
+	1    1550 4600
 	1    0    0    -1
 $EndComp
@@
 L power:GND #PWR0107
 U 1 1 5CCACD7C
-P 14150 9100
-F 0 "#PWR0107" H 14150 8850 50  0001 C CNN
-F 1 "GND" H 14155 8927 50  0000 C CNN
-F 2 "" H 14150 9100 50  0001 C CNN
-F 3 "" H 14150 9100 50  0001 C CNN
-	1    14150 9100
+P 10800 8500
+F 0 "#PWR0107" H 10800 8250 50  0001 C CNN
+F 1 "GND" H 10805 8327 50  0000 C CNN
+F 2 "" H 10800 8500 50  0001 C CNN
+F 3 "" H 10800 8500 50  0001 C CNN
+	1    10800 8500
 	1    0    0    -1
 $EndComp
@@
 	1450 2400 4000 2400
 Wire Wire Line
-	4000 4050 4550 4050
-Wire Wire Line
-	4000 4150 4550 4150
-Wire Wire Line
-	4000 4250 4550 4250
-Wire Wire Line
-	4000 4350 4550 4350
+	4000 4050 5050 4050
+Wire Wire Line
+	4000 4150 5050 4150
+Wire Wire Line
+	4000 4250 5050 4250
+Wire Wire Line
+	4000 4350 5050 4350
 Wire Wire Line
 	12300 1700 12300 1800
-$Comp
-L power:+3V3 #+3V0101
-U 1 1 60274272
-P 11300 1800
-F 0 "#+3V0101" H 11300 1800 50  0001 C CNN
-F 1 "+3V3" V 11200 1600 59  0000 L BNN
-F 2 "" H 11300 1800 50  0001 C CNN
-F 3 "" H 11300 1800 50  0001 C CNN
-	1    11300 1800
-	1    0    0    -1
-$EndComp
 Wire Wire Line
 	10900 2200 11600 2200
@@
 BLANK
 Wire Wire Line
-	11300 1800 11300 2100
+	11300 1700 11300 2100
 NoConn ~ 11600 3000
 NoConn ~ 11600 3600
@@
 P 3800 4250
 F 0 "RN1" V 3383 4250 50  0000 C CNN
-F 1 "R_Pack04" V 3474 4250 50  0000 C CNN
+F 1 "1K" V 3474 4250 50  0000 C CNN
 F 2 "Resistor_SMD:R_Array_Convex_4x0603" V 4075 4250 50  0001 C CNN
 F 3 "~" H 3800 4250 50  0001 C CNN
@@
 Wire Wire Line
 	2600 4400 1450 4400
+Text Label 10950 2200 0    50   ~ 0
+IREF
+Text Label 14400 1700 0    50   ~ 0
+OUT0
+Text Label 14400 2000 0    50   ~ 0
+OUT1
+Text Label 14400 2300 0    50   ~ 0
+OUT2
+Text Label 14400 2600 0    50   ~ 0
+OUT3
+Text Label 14400 2900 0    50   ~ 0
+OUT4
+Text Label 14400 3200 0    50   ~ 0
+OUT5
+Text Label 14400 3500 0    50   ~ 0
+OUT6
+Text Label 14400 3800 0    50   ~ 0
+OUT7
+Text Label 14400 4100 0    50   ~ 0
+OUT8
+Text Label 14400 4400 0    50   ~ 0
+OUT9
+Text Label 14400 4700 0    50   ~ 0
+OUT10
+Text Label 14400 5000 0    50   ~ 0
+OUT11
+Text Label 14400 5300 0    50   ~ 0
+OUT12
+Text Label 14400 5600 0    50   ~ 0
+OUT13
+Text Label 14400 5900 0    50   ~ 0
+OUT14
+Text Label 14400 6200 0    50   ~ 0
+OUT15
+Text Label 11050 7700 0    50   ~ 0
+OUT15S
+Text Label 1900 3200 0    50   ~ 0
+ST-IN
+Text Label 1900 3600 0    50   ~ 0
+TH-IN
+Text Label 1900 4000 0    50   ~ 0
+AUX-IN
+Text Label 1900 4400 0    50   ~ 0
+OUT-ISP-OUT
+$Comp
+L power:+3V3 #PWR0109
+U 1 1 60242FCF
+P 6000 2100
+F 0 "#PWR0109" H 6000 1950 50  0001 C CNN
+F 1 "+3V3" H 6015 2273 50  0000 C CNN
+F 2 "" H 6000 2100 50  0001 C CNN
+F 3 "" H 6000 2100 50  0001 C CNN
+	1    6000 2100
+	1    0    0    -1
+$EndComp
+$Comp
+L power:+3V3 #PWR0112
+U 1 1 6024C267
+P 11300 1700
+F 0 "#PWR0112" H 11300 1550 50  0001 C CNN
+F 1 "+3V3" H 11315 1873 50  0000 C CNN
+F 2 "" H 11300 1700 50  0001 C CNN
+F 3 "" H 11300 1700 50  0001 C CNN
+	1    11300 1700
+	1    0    0    -1
+$EndComp
+$Comp
+L power:+3V3 #PWR0113
+U 1 1 6024D34E
+P 12300 1700
+F 0 "#PWR0113" H 12300 1550 50  0001 C CNN
+F 1 "+3V3" H 12315 1873 50  0000 C CNN
+F 2 "" H 12300 1700 50  0001 C CNN
+F 3 "" H 12300 1700 50  0001 C CNN
+	1    12300 1700
+	1    0    0    -1
+$EndComp
+$Comp
+L power:+3V3 #PWR0114
+U 1 1 6025D63E
+P 5700 6150
+F 0 "#PWR0114" H 5700 6000 50  0001 C CNN
+F 1 "+3V3" H 5715 6323 50  0000 C CNN
+F 2 "" H 5700 6150 50  0001 C CNN
+F 3 "" H 5700 6150 50  0001 C CNN
+	1    5700 6150
+	1    0    0    -1
+$EndComp
 $EndSCHEMATC

Commit message: Add TSSOP 20 versions
Other:
- note added: "NXP LPC812\nARM Cortex-M0\n16K Flash, 4K RAM\nXSON-16"
- note removed: "NXP LPC812\nARM Cortex-M0\n16K Flash, 4K RAM\nTSSOP-16"
Changed lines of the file:
@@
 Sheet 1 1
 Title "DIY RC Light Controller Mk4 Rev4"
-Date "2019-05-01"
+Date "2021-02-11"
 Rev "4"
 Comp "LANE Boys RC"
@@
 X5R or X7R
 Text Notes 6800 8400 0    59   ~ 0
-NXP LPC812\nARM Cortex-M0\n16K Flash, 4K RAM\nTSSOP-16
+NXP LPC812\nARM Cortex-M0\n16K Flash, 4K RAM\nXSON-16
 Text Notes 9950 7300 0    85   ~ 0
 Switched output\nfor light bar or similar
