File: preprocessor/electronics-multi-aux/XSON16-version/preprocessor-multi-aux-xson16.kicad_pcb (KiCad board)
At the start: 2 copper layers, 17 x 24 mm, 16 parts, among them P1 ST-IN, P2 ST-OUT, P3 TH-IN, P4 TH-OUT, P5 AUX-IN, P6 LIGHT CONTROLLER, P7 AUX2-IN, P8 AUX3-IN, U1 MCP1703T-3302E/CB, U2 LPC812M101JTB16_XSON16

Commit message: Tweak layout
Parts:
- moved RN1 0.41 mm to (125.6, 62.0)
- moved R7 0.25 mm to (129.1, 62.0)
Routing:
- net /ST: track 7.10 -> 6.50 mm
- net /AUX_IN: track 9.65 -> 9.07 mm
- net /AUX2_IN: track 8.87 -> 8.34 mm

Commit message: Add TSSOP 20 versions
Other:
- board text added: "3ch-PP LANE Boys RC"
