File: preprocessor/electronics/TSSOP20-version/preprocessor.sch (KiCad schematic (older format))
At the start: 11 parts, among them P1 ST-IN, P2 ST-OUT, P3 TH-IN, P4 TH-OUT, P5 AUX-IN, P6 LIGHT CONTROLLER, U1 MCP1703T-3302E/CB, U2 LPC811M001JDH16_TSSOP16

Commit message: Add TSSOP 20 versions
Parts:
- U2: value LPC811M001JDH16_TSSOP16 -> LPC812M001JDH20_TSSOP20; footprint Package_SON:NXP_XSON-16 -> Package_SO:TSSOP-20_4.4x6.5mm_P0.65mm; symbol MCU_NXP_LPC:LPC812M101JTB16 -> MCU_NXP_LPC:LPC812M101JDH20
Connections:
- wire segments 65 -> 63
- no-connect marks 10 -> 14
Other:
- moved on the sheet: P6, RN1
Changed lines of the file:
@@
 Title "Pre-processor for RC Light Controller"
 Date "2021-02-11"
-Rev "4"
+Rev "5"
 Comp "LANE Boys RC"
-Comment1 "XSON16 package due to TSSOP16 shortage in 2021"
+Comment1 "TSSOP20 package due to TSSOP16 shortage in 2021"
 Comment2 ""
 Comment3 ""
@@
 $EndDescr
 $Comp
-L MCU_NXP_LPC:LPC812M101JTB16 U2
+L MCU_NXP_LPC:LPC812M101JDH20 U2
 U 1 1 58AF9BA8
 P 7300 2550
 F 0 "U2" H 7200 2650 10  0001 C CNN
-F 1 "LPC811M001JDH16_TSSOP16" H 8000 3100 60  0000 C CNN
-F 2 "Package_SON:NXP_XSON-16" H 7200 2650 60  0001 C CNN
+F 1 "LPC812M001JDH20_TSSOP20" H 8050 3200 60  0000 C CNN
+F 2 "Package_SO:TSSOP-20_4.4x6.5mm_P0.65mm" H 7200 2650 60  0001 C CNN
 F 3 "" H 7200 2650 60  0000 C CNN
 	1    7300 2550
@@
 L Connector_Generic:Conn_01x03 P6
 U 1 1 58AF9DBB
-P 5400 4800
-F 0 "P6" H 5400 5000 50  0000 C CNN
-F 1 "LIGHT CONTROLLER" V 5500 4800 50  0000 C CNN
-F 2 "Pin_Headers:Pin_Header_Straight_1x03_Pitch2.54mm" H 5400 4800 50  0001 C CNN
-F 3 "" H 5400 4800 50  0000 C CNN
-	1    5400 4800
+P 5250 5250
+F 0 "P6" H 5250 5450 50  0000 C CNN
+F 1 "LIGHT CONTROLLER" V 5350 5250 50  0000 C CNN
+F 2 "Pin_Headers:Pin_Header_Straight_1x03_Pitch2.54mm" H 5250 5250 50  0001 C CNN
+F 3 "" H 5250 5250 50  0000 C CNN
+	1    5250 5250
 	1    0    0    1
 $EndComp
@@
 L power:VCC #PWR010
 U 1 1 58AFAD17
-P 5100 4500
-F 0 "#PWR010" H 5100 4350 50  0001 C CNN
-F 1 "VCC" H 5100 4650 50  0000 C CNN
-F 2 "" H 5100 4500 50  0000 C CNN
-F 3 "" H 5100 4500 50  0000 C CNN
-	1    5100 4500
+P 4950 4950
+F 0 "#PWR010" H 4950 4800 50  0001 C CNN
+F 1 "VCC" H 4950 5100 50  0000 C CNN
+F 2 "" H 4950 4950 50  0000 C CNN
+F 3 "" H 4950 4950 50  0000 C CNN
+	1    4950 4950
 	1    0    0    -1
 $EndComp
@@
 L power:GND #PWR011
 U 1 1 58AFADBD
-P 5100 5000
-F 0 "#PWR011" H 5100 4750 50  0001 C CNN
-F 1 "GND" H 5100 4850 50  0000 C CNN
-F 2 "" H 5100 5000 50  0000 C CNN
-F 3 "" H 5100 5000 50  0000 C CNN
-	1    5100 5000
-	1    0    0    -1
-$EndComp
-Wire Wire Line
-	5200 4800 5100 4800
-Wire Wire Line
-	5100 4800 5100 4500
-Wire Wire Line
-	5200 4900 5100 4900
-Wire Wire Line
-	5100 4900 5100 5000
+P 4950 5450
+F 0 "#PWR011" H 4950 5200 50  0001 C CNN
+F 1 "GND" H 4950 5300 50  0000 C CNN
+F 2 "" H 4950 5450 50  0000 C CNN
+F 3 "" H 4950 5450 50  0000 C CNN
+	1    4950 5450
+	1    0    0    -1
+$EndComp
+Wire Wire Line
+	5050 5250 4950 5250
+Wire Wire Line
+	4950 5250 4950 4950
+Wire Wire Line
+	5050 5350 4950 5350
+Wire Wire Line
+	4950 5350 4950 5450
 Wire Wire Line
 	2850 1950 3450 1950
 Wire Wire Line
 	2850 2950 3450 2950
-NoConn ~ 8000 2450
 NoConn ~ 8000 2650
 NoConn ~ 8000 2350
 NoConn ~ 6600 2350
 NoConn ~ 6600 2450
-NoConn ~ 6600 2550
 NoConn ~ 6600 2750
 NoConn ~ 6600 2850
-NoConn ~ 8000 2550
 Wire Wire Line
 	2850 2450 3450 2450
@@
 	3400 1500 3100 1500
 Connection ~ 3100 1500
-Text Label 3650 3900 0    50   ~ 0
+Text Label 4050 3900 2    50   ~ 0
 AUX_IN
-Text Label 3650 2950 0    50   ~ 0
+Text Label 4050 2950 2    50   ~ 0
 TH_IN
-Text Label 3650 1950 0    50   ~ 0
+Text Label 4050 1950 2    50   ~ 0
 ST_IN
 Text Label 3750 6400 0    60   ~ 0
 3V3
 Wire Wire Line
-	2850 3900 4600 3900
+	2850 3900 4050 3900
 $Comp
 L power:PWR_FLAG #FLG013
@@
 L Device:R_Pack04 RN1
 U 1 1 601F9E94
-P 4800 3900
-F 0 "RN1" V 4383 3900 50  0000 C CNN
-F 1 "1K" V 4474 3900 50  0000 C CNN
-F 2 "Resistor_SMD:R_Array_Convex_4x0603" V 5075 3900 50  0001 C CNN
-F 3 "~" H 4800 3900 50  0001 C CNN
-	1    4800 3900
+P 5350 3900
+F 0 "RN1" V 4933 3900 50  0000 C CNN
+F 1 "1K" V 5024 3900 50  0000 C CNN
+F 2 "Resistor_SMD:R_Array_Convex_4x0603" V 5625 3900 50  0001 C CNN
+F 3 "~" H 5350 3900 50  0001 C CNN
+	1    5350 3900
 	0    1    1    0
 $EndComp
@@
 	7300 1850 7300 1950
 Wire Wire Line
-	3450 2950 3950 2950
-Wire Wire Line
-	3950 2950 3950 3800
-Wire Wire Line
-	3950 3800 4600 3800
+	3450 2950 4050 2950
 Connection ~ 3450 2950
-Wire Wire Line
-	4050 3700 4600 3700
-Wire Wire Line
-	4050 1950 4050 3700
-Wire Wire Line
-	4600 4000 3500 4000
-Text Label 3650 4000 0    50   ~ 0
+Text Label 4250 5150 0    50   ~ 0
 LIGHT_OUT
 Wire Wire Line
-	5000 3700 5600 3700
-Text Label 5600 3700 2    50   ~ 0
+	5550 3700 6150 3700
+Text Label 6150 3700 2    50   ~ 0
 ST
 Wire Wire Line
-	5000 3800 5600 3800
-Text Label 5600 3800 2    50   ~ 0
+	5550 3800 6150 3800
+Text Label 6150 4000 2    50   ~ 0
 TH
 Wire Wire Line
-	5000 3900 5600 3900
-Text Label 5600 3900 2    50   ~ 0
+	5550 3900 6150 3900
+Text Label 6150 3800 2    50   ~ 0
 AUX
 Wire Wire Line
-	5000 4000 5600 4000
-Text Label 5600 4000 2    50   ~ 0
+	5550 4000 6150 4000
+Text Label 6150 3900 2    50   ~ 0
 LIGHT
 Wire Wire Line
@@
 	2000 6400 2550 6400
 Wire Wire Line
-	6150 2250 6600 2250
-Text Label 6150 2250 0    50   ~ 0
+	6150 2150 6600 2150
+Text Label 6150 2150 0    50   ~ 0
 ST
 Wire Wire Line
-	6150 2650 6600 2650
-Text Label 6150 2650 0    50   ~ 0
+	6150 2550 6600 2550
+Text Label 6150 2550 0    50   ~ 0
 TH
 Wire Wire Line
-	8000 2750 8500 2750
-Text Label 8500 2750 2    50   ~ 0
+	8000 2450 8500 2450
+Text Label 8500 2450 2    50   ~ 0
 LIGHT
 Wire Wire Line
-	8000 2850 8500 2850
-Text Label 8500 2850 2    50   ~ 0
+	8000 2550 8500 2550
+Text Label 8500 2550 2    50   ~ 0
 AUX
 NoConn ~ 8000 2250
 Wire Wire Line
-	3500 4000 3500 4700
-Wire Wire Line
-	3500 4700 5200 4700
+	4250 5150 5050 5150
+NoConn ~ 6600 2950
+NoConn ~ 8000 2150
+NoConn ~ 8000 2750
+NoConn ~ 8000 2850
+NoConn ~ 8000 2950
+NoConn ~ 6600 2650
+NoConn ~ 6600 2250
+Wire Wire Line
+	4700 3700 5150 3700
+Wire Wire Line
+	4700 3800 5150 3800
+Wire Wire Line
+	4700 3900 5150 3900
+Wire Wire Line
+	4700 4000 5150 4000
+Text Label 4700 3800 0    50   ~ 0
+AUX_IN
+Text Label 4700 4000 0    50   ~ 0
+TH_IN
+Text Label 4700 3900 0    50   ~ 0
+LIGHT_OUT
+Text Label 4700 3700 0    50   ~ 0
+ST_IN
 $EndSCHEMATC
