File: preprocessor/electronics/TSSOP20-version/preprocessor.kicad_pcb (KiCad board)
At the start: 2 copper layers, 17 x 17 mm, 11 parts, among them P1 ST-IN, P2 ST-OUT, P3 TH-IN, P4 TH-OUT, P5 AUX-IN, P6 LIGHT CONTROLLER, U1 MCP1703T-3302E/CB, U2 LPC812M001JDH20_TSSOP20

Commit message: Add product and LANE Boys RC label
Other:
- board text added: "3ch-PP LANE Boys RC"
