File: preprocessor/electronics/XSON16-version/preprocessor.kicad_pcb (KiCad board)
At the start: 2 copper layers, 17 x 17 mm, 11 parts, among them P1 ST-IN, P2 ST-OUT, P3 TH-IN, P4 TH-OUT, P5 AUX-IN, P6 LIGHT CONTROLLER, U1 MCP1703T-3302E/CB, U2 LPC811M001JDH16_TSSOP16

Commit message: Add and fix product label on silkscreen
Other:
- board text added: "3ch-PP LANE Boys RC"

Commit message: Clear solder paste reduction and add Gerber
Other:
- rule pad_to_mask_clearance: 0.0508 -> 0
Changed lines of the file:
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@@
     (pad_size 0.8 0.4)
     (pad_drill 0)
-    (pad_to_mask_clearance 0.0508)
-    (solder_mask_min_width 0.0508)
-    (pad_to_paste_clearance_ratio -0.05)
+    (pad_to_mask_clearance 0)
     (aux_axis_origin 114.3 66.04)
     (grid_origin 114.3 66.04)
     (visible_elements 7FFFFF7F)
     (pcbplotparams
-      (layerselection 0x010f0_ffffffff)
-      (usegerberextensions true)
+      (layerselection 0x010f8_ffffffff)
+      (usegerberextensions false)
       (usegerberattributes false)
       (usegerberadvancedattributes false)
@@
       (effects (font (size 0.5 0.5) (thickness 0.08)))
     )
-    (pad 1 smd roundrect (at -1.025 0 270) (size 1.15 1.4) (layers F.Cu F.Paste F.Mask) (roundrect_rratio 0.217391)
-      (net 1 VCC))
-    (pad 2 smd roundrect (at 1.025 0 270) (size 1.15 1.4) (layers F.Cu F.Paste F.Mask) (roundrect_rratio 0.217391)
+    (pad 1 smd roundrect (at -1.025 0 270) (size 1.15 1.4) (layers F.Cu F.Paste F.Mask) (roundrect_rratio 0.2173904347826087)
+      (net 1 VCC))
+    (pad 2 smd roundrect (at 1.025 0 270) (size 1.15 1.4) (layers F.Cu F.Paste F.Mask) (roundrect_rratio 0.2173904347826087)
       (net 2 GND))
     (model ${KISYS3DMOD}/Capacitor_SMD.3dshapes/C_0805_2012Metric.wrl
@@
       (effects (font (size 0.5 0.5) (thickness 0.08)))
     )
-    (pad 2 smd roundrect (at 1.025 0 90) (size 1.15 1.4) (layers F.Cu F.Paste F.Mask) (roundrect_rratio 0.217391)
-      (net 2 GND))
-    (pad 1 smd roundrect (at -1.025 0 90) (size 1.15 1.4) (layers F.Cu F.Paste F.Mask) (roundrect_rratio 0.217391)
+    (pad 2 smd roundrect (at 1.025 0 90) (size 1.15 1.4) (layers F.Cu F.Paste F.Mask) (roundrect_rratio 0.2173904347826087)
+      (net 2 GND))
+    (pad 1 smd roundrect (at -1.025 0 90) (size 1.15 1.4) (layers F.Cu F.Paste F.Mask) (roundrect_rratio 0.2173904347826087)
       (net 3 +3V3))
     (model ${KISYS3DMOD}/Capacitor_SMD.3dshapes/C_0805_2012Metric.wrl
@@
   )
   (zone (net 2) (net_name GND) (layer B.Cu) (hatch edge 0.508)
-    (connect_pads (clearance 0.254))
-    (min_thickness 0.254)
+    (connect_pads (clearance 0.2032))
+    (min_thickness 0.1524)
     (fill yes (arc_segments 16) (thermal_gap 0.254) (thermal_bridge_width 0.3048))
     (polygon
