File: mk4-tlc5940-lpc812/electronics/pcb-size-27x20/rc-light-controller-tlc5940-lpc812.sch (KiCad schematic (older format))
At the start: 42 parts, among them T1 NMOSSOT23, U2 TLC5940PWP

Commit message: Fix R5, T1, U$1 not being reflected in Pick and Place file
Parts:
- renumbered R6 to R5
Changed lines of the file:
@@
 $EndComp
 $Comp
-L rc-light-controller-tlc5940-lpc812-eagle-import:R-EU_R0603 R6
+L rc-light-controller-tlc5940-lpc812-eagle-import:R-EU_R0603 R5
 U 1 1 5049E5A2
 P 2450 4000
-F 0 "R6" H 2300 4059 59  0000 L BNN
+F 0 "R5" H 2300 4059 59  0000 L BNN
 F 1 "1k" H 2300 3870 59  0000 L BNN
 F 2 "Resistor_SMD:R_0603_1608Metric" H 2450 4000 50  0001 C CNN
