File: mk4-tlc5940-lpc812/electronics-switching/LPC832-TSSOP20-version/rc-light-controller-switching-lpc832.kicad_pcb (KiCad board)
At the start: 2 copper layers, 44 x 23 mm, 20 parts, among them J1 Pinheader right-angle 2x17, J2 Pinheader straight 1x06, J3 Pinheader straight 1x06, T1 PMV30UN, T2 PMV30UN, T3 PMV30UN, T4 PMV30UN, T5 PMV30UN, T6 PMV30UN, T7 PMV30UN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

Commit message: Fix soldermask settings
Other:
- rule pad_to_mask_clearance: 0.0254 -> 0
