File: mk4-tlc5940-lpc812/tools/webusb-programmer/rev3-ch552/electronics/webusb-programmer-ch552.kicad_pcb (KiCad board)
At the start: 2 copper layers, 38 x 20 mm, 19 parts, among them J1 Light Controller, J2 USB_B_Micro, U1 STMPS2141STR, U2 CH552G

Commit message: Improve fab layer
Parts:
- D1: value LC POWER -> Blue
- D2: value OK -> Green
- D3: value BUSY -> Amber
- D4: value ERROR -> Red
- D5: value MCU POWER -> White

Commit message: Update schematics to reflect green LED being low brightness
Parts:
- D1: value Blue -> B
- D2: value Green -> G
- D3: value Amber -> Y
- D4: value Red -> R
- D5: value White -> W
- R3: value 2k7 -> 180
