File: mk4-tlc5940-lpc812/tools/webusb-programmer/rev4-ch551-ch552/electronics/webusb-programmer-ch551-ch552.sch (KiCad schematic (older format))
At the start: 19 parts, among them J1 Light Controller, J2 USB_B_Micro, U1 TC118S, U2 CH552G or CH551G

Commit message: Improve naming of project specific schematics component library
Parts:
- U1: symbol wla-atsamd21:TC118S -> wla-project-specific-components:TC118S
- U2: symbol wla-atsamd21:CH552G -> wla-project-specific-components:CH552G
Changed lines of the file:
@@
 Blue
 $Comp
-L wla-atsamd21:CH552G U2
+L wla-project-specific-components:CH552G U2
 U 1 1 604D2755
 P 3800 6050
@@
 ~OK
 $Comp
-L wla-atsamd21:TC118S U1
+L wla-project-specific-components:TC118S U1
 U 1 1 6180984C
 P 7300 1700

Commit message: Remove series resistor, TC118S motor driver does not need it
Parts:
- removed R1: 1R, Resistor_SMD:R_0603_1608Metric_Pad0.98x0.95mm_HandSolder, symbol Device:R
- renumbered R2 to R1, R3 to R2, R4 to R3, R5 to R4
Connections:
- net VLIGHT: now also U1.5 (OUTB)
Other:
- note added: "The LEDs are conneced at the cathode\nto prevent them from lighting\nup after power up before the software\ncan initialize the ports (pull-up by default)\nError and Busy use the same resistor value, \nand since they never light up together we \ncan share one resistor. \nOK (green) uses a different technology \nso needs its own resistor."
- note removed: "The LEDs are conneced at the cathode\nto prevent them from lighting\nup after power up before the software\ncan initialize the ports (pull-up by default)\nError and Busy use the same resistor value, \nand since they never light up together we \ncan share one resistor. \nOK (green) behaves differently so needs \nits own resistor."
Changed lines of the file:
@@
 	5250 3000 5250 3250
 $Comp
-L Device:R R5
+L Device:R R4
 U 1 1 5E6FD675
 P 5250 2450
-F 0 "R5" H 5320 2496 50  0000 L CNN
+F 0 "R4" H 5320 2496 50  0000 L CNN
 F 1 "1k8" H 5320 2405 50  0000 L CNN
 F 2 "Resistor_SMD:R_0603_1608Metric_Pad1.05x0.95mm_HandSolder" V 5180 2450 50  0001 C CNN
@@
 $EndComp
 Text Notes 3300 1800 0    50   ~ 0
-The LEDs are conneced at the cathode\nto prevent them from lighting\nup after power up before the software\ncan initialize the ports (pull-up by default)\nError and Busy use the same resistor value, \nand since they never light up together we \ncan share one resistor. \nOK (green) behaves differently so needs \nits own resistor.
+The LEDs are conneced at the cathode\nto prevent them from lighting\nup after power up before the software\ncan initialize the ports (pull-up by default)\nError and Busy use the same resistor value, \nand since they never light up together we \ncan share one resistor. \nOK (green) uses a different technology \nso needs its own resistor.
 $Comp
 L Connector:TestPoint TP1
@@
 	3500 2600 3500 2700
 $Comp
-L Device:R R3
+L Device:R R2
 U 1 1 5E6FABAC
 P 3500 2450
-F 0 "R3" H 3570 2496 50  0000 L CNN
+F 0 "R2" H 3570 2496 50  0000 L CNN
 F 1 "180" H 3570 2405 50  0000 L CNN
 F 2 "Resistor_SMD:R_0603_1608Metric_Pad1.05x0.95mm_HandSolder" V 3430 2450 50  0001 C CNN
@@
 $EndComp
 $Comp
-L Device:R R4
+L Device:R R3
 U 1 1 5E6FC0B8
 P 4700 2450
-F 0 "R4" H 4770 2496 50  0000 L CNN
+F 0 "R3" H 4770 2496 50  0000 L CNN
 F 1 "1k2" H 4770 2405 50  0000 L CNN
 F 2 "Resistor_SMD:R_0603_1608Metric_Pad1.05x0.95mm_HandSolder" V 4630 2450 50  0001 C CNN
@@
 	1    0    0    -1
 $EndComp
-Wire Wire Line
-	7750 1800 8300 1800
 NoConn ~ 7750 1600
 $Comp
@@
 Motor driver IC used\nas power switch for \nthe light controller\n\nINA INB OUTA OUTB \nL    L  Hi-Z  Hi-Z\nH    L   H    L\nL    H   L    H\nH    H   L    L
 $Comp
-L Device:R R2
+L Device:R R1
 U 1 1 5E6FD03E
 P 9250 2050
-F 0 "R2" H 9320 2096 50  0000 L CNN
+F 0 "R1" H 9320 2096 50  0000 L CNN
 F 1 "1k8" H 9320 2005 50  0000 L CNN
 F 2 "Resistor_SMD:R_0603_1608Metric_Pad1.05x0.95mm_HandSolder" V 9180 2050 50  0001 C CNN
@@
 	1    0    0    -1
 $EndComp
-$Comp
-L Device:R R1
-U 1 1 6183E54C
-P 8450 1800
-F 0 "R1" H 8520 1846 50  0000 L CNN
-F 1 "1R" H 8520 1755 50  0000 L CNN
-F 2 "Resistor_SMD:R_0603_1608Metric_Pad0.98x0.95mm_HandSolder" V 8380 1800 50  0001 C CNN
-F 3 "~" H 8450 1800 50  0001 C CNN
-	1    8450 1800
-	0    1    1    0
-$EndComp
-Wire Wire Line
-	8600 1800 9250 1800
+Wire Wire Line
+	7750 1800 9250 1800
 $EndSCHEMATC

Commit message: Add BOM for WebUSB Programmer Rev4
Parts:
- U1: LCSC part number (none) -> C88308
- U2: LCSC part number (none) -> C111292
Changed lines of the file:
@@
 F 2 "Package_SO:SO-16_3.9x9.9mm_P1.27mm" H 2200 6000 50  0001 C CNN
 F 3 "" H 2200 6000 50  0001 C CNN
+F 4 "C111292" H 3800 6050 50  0001 C CNN "LCSC part number"
 	1    3800 6050
 	1    0    0    -1
@@
 F 1 "TC118S" H 7600 1350 50  0000 C CNN
 F 2 "Package_SO:SOP-8_3.9x4.9mm_P1.27mm" H 7300 1700 50  0001 C CNN
-F 3 "LCSC C88308" H 7300 1700 50  0001 C CNN
+F 3 "" H 7300 1700 50  0001 C CNN
+F 4 "C88308" H 7300 1700 50  0001 C CNN "LCSC part number"
 	1    7300 1700
 	1    0    0    -1

Commit message: Make C1 on WebUSB 10uF to combat voltage drop when light controller is turned on
Parts:
- C1: value 1u -> 10u
Other:
- note added: "C1 needs to be rather large, \nbecause when the Light Controller \nis powered up the 47uF needs to \nbe charged, causing a voltage \ndrop that could crash the WebUSB \nprogrammer -- especially when \nusing longer USB cables."
Changed lines of the file:
@@
 Sheet 1 1
 Title "WebUSB Programmer for Light Controller Mk4"
-Date "2021-10-30"
+Date "2022-03-24"
 Rev "4"
 Comp "LANE Boys RC"
@@
 P 3300 4950
 F 0 "C1" H 3415 4996 50  0000 L CNN
-F 1 "1u" H 3415 4905 50  0000 L CNN
+F 1 "10u" H 3415 4905 50  0000 L CNN
 F 2 "Capacitor_SMD:C_0603_1608Metric" H 3338 4800 50  0001 C CNN
 F 3 "~" H 3300 4950 50  0001 C CNN
@@
 Wire Wire Line
 	7750 1800 9250 1800
+Text Notes 1700 5050 0    50   ~ 0
+C1 needs to be rather large, \nbecause when the Light Controller \nis powered up the 47uF needs to \nbe charged, causing a voltage \ndrop that could crash the WebUSB \nprogrammer -- especially when \nusing longer USB cables.
 $EndSCHEMATC
