File: mk4-tlc5940-lpc812/electronics/LPC832-TSSOP20-SBUS-version/rc-light-controller-tlc5940-lpc832-sbus.kicad_pcb (KiCad board)
At the start: 2 copper layers, 29 x 18 mm, 36 parts, among them Q1 2N7002K, Q2 NMOSSOT23, U1 3V3, U2 LPC832M101FDH20, U3 TLC5940PWP

Commit message: Improve schematics and layout
Routing:
- net GND: track 1.74 -> 1.14 mm, vias 23 -> 24
