File: mk4-tlc5940-lpc812/electronics/LPC832-TSSOP20-SBUS-version/rc-light-controller-tlc5940-lpc832-sbus.sch (KiCad schematic (older format))
At the start: 36 parts, among them Q1 2N7002K, Q2 NMOSSOT23, U1 3V3, U2 LPC832M101FDH20, U3 TLC5940PWP

Commit message: Improve schematics and layout
Other:
- note added: "Important: this MOSFET needs to have\na low gate capacitance (~20pf), as otherwise\nit will distort the UART / Servo signal"
- note added: "LDO: \nMCP1702, MCP1703\nME6209A33M3G"
- note added: "N-Channel MOSFET\nSOT23 package\ne.g. PMV16UN, PMV30UN, \nSI2302. AO3400, DMN2075U-7"
- note added: "S.BUS inverter"
- note removed: "LDO: Microchip \nMCP1702 or MCP1703"
- note removed: "N-Channel MOSFET\nSOT23 package\ne.g. NXP PMV16UN"
- moved on the sheet: C3, OUT15S1, Q1, Q2, R2, U2

Commit message: Fix help text in schematics
Other:
- note added: "Important: this MOSFET needs to have\na low gate capacitance (~~20pf), as otherwise\nit will distort the UART / Servo signal"
- note added: "Special pins:\nPIO0_0 (19) ISP UART RX\nPIO0_4 ( 6) ISP UART TX\nPIO0_5 ( 5) RESET\nPIO0_10 (10) Open drain\nPIO0_11 ( 9) Open drain\nPIO0_2 ( 8) SWDIO\nPIO0_3 ( 7) SWCLK"
- note removed: "Important: this MOSFET needs to have\na low gate capacitance (~20pf), as otherwise\nit will distort the UART / Servo signal"
- note removed: "Special pins:\nPIO0_0 (16) ISP UART RX\nPIO0_4 ( 4) ISP UART TX\nPIO0_5 ( 3) RESET\nPIO0_10 ( 8) Open drain\nPIO0_11 ( 7) Open drain\nPIO0_2 ( 6) SWDIO\nPIO0_3 ( 5) SWCLK"
Changed lines of the file:
@@
 $EndComp
 Text Notes 3150 9850 0    56   ~ 0
-Special pins:\nPIO0_0  (16)   ISP UART RX\nPIO0_4  ( 4)   ISP UART TX\nPIO0_5  ( 3)   RESET\nPIO0_10 ( 8)   Open drain\nPIO0_11 ( 7)   Open drain\nPIO0_2  ( 6)   SWDIO\nPIO0_3  ( 5)   SWCLK
+Special pins:\nPIO0_0  (19)   ISP UART RX\nPIO0_4  ( 6)   ISP UART TX\nPIO0_5  ( 5)   RESET\nPIO0_10 (10)   Open drain\nPIO0_11 ( 9)   Open drain\nPIO0_2  ( 8)   SWDIO\nPIO0_3  ( 7)   SWCLK
 Text Notes 1050 2000 0    85   ~ 0
 Servo in/out
@@
 	4050 4050 5050 4050
 Text Notes 8700 6850 0    50   ~ 0
-Important: this MOSFET needs to have\na low gate capacitance (~20pf), as otherwise\nit will distort the UART / Servo signal
+Important: this MOSFET needs to have\na low gate capacitance (~~20pf), as otherwise\nit will distort the UART / Servo signal
 Wire Wire Line
 	5550 7700 6650 7700
