File: mk4-tlc5940-lpc812/tools/webusb-programmer/rev6-ch551-ch552-ch554/electronics/webusb-programmer-rev6.kicad_pcb (KiCad board)
At the start: 2 copper layers, 38 x 20 mm, 18 parts, among them J1 Light Controller, J2 USB_C_Receptacle_USB2.0, U1 TC118S, U2 CH552G

Commit message: WebUSB rev 6 for production
Parts:
- D6: footprint Diode_SMD:D_SOD-123F -> Diode_SMD:D_SOD-123
