File: mk4-tlc5940-lpc812/tools/webusb-programmer/rev6-ch551-ch552-ch554/electronics/webusb-programmer-rev6.kicad_sch (KiCad schematic)
At the start: 18 parts, among them J1 Light Controller, J2 USB_C_Receptacle_USB2.0, U1 TC118S, U2 CH552G

Commit message: WebUSB rev 6 for production
Parts:
- D6: footprint Diode_SMD:D_SOD-123F -> Diode_SMD:D_SOD-123
Changed lines of the file:
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@@
       (effects (font (size 1.27 1.27)) (justify right))
     )
-    (property "Footprint" "Diode_SMD:D_SOD-123F" (id 2) (at 92.71 113.03 0)
+    (property "Footprint" "Diode_SMD:D_SOD-123" (id 2) (at 92.71 113.03 0)
       (effects (font (size 1.27 1.27)) hide)
     )
@@
     )
     (path "/a7bb18ee-f118-4fbc-b69e-bcab853f2f90"
-      (reference "D6") (unit 1) (value "B5819WS") (footprint "Diode_SMD:D_SOD-123F")
+      (reference "D6") (unit 1) (value "B5819WS") (footprint "Diode_SMD:D_SOD-123")
     )
     (path "/00000000-0000-0000-0000-00005e6fe83d"
