File: mk4-tlc5940-lpc812/electronics-pinheader/rev4/rc-light-controller-pinheader.kicad_sch (KiCad schematic)
At the start: 14 parts, among them J1 Pinheader right-angle 2x17, J2 Pinheader straight 1x06, J3 Pinheader straight 1x06, T9 PMV30UN, U1 LPC832M101FDH20, U2 TLC5940PWP, U3 MCP1703A-3302_SOT23

Commit message: Improve filenames and update Gerbers
Parts:
- U1: value LPC832M101FDH20 -> LPC824M201FDH20
Changed lines of the file:
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@@
     (in_bom yes) (on_board yes)
     (property "Reference" "U1" (id 0) (at 212.09 191.77 0))
-    (property "Value" "LPC832M101FDH20" (id 1) (at 182.88 191.77 0))
+    (property "Value" "LPC824M201FDH20" (id 1) (at 182.88 191.77 0))
     (property "Footprint" "Package_SO:TSSOP-20_4.4x6.5mm_P0.65mm" (id 2) (at 224.79 190.5 0)
       (effects (font (size 1.27 1.27)) hide)
@@
     )
     (path "/00000000-0000-0000-0000-000060608195"
-      (reference "U1") (unit 1) (value "LPC832M101FDH20") (footprint "Package_SO:TSSOP-20_4.4x6.5mm_P0.65mm")
+      (reference "U1") (unit 1) (value "LPC824M201FDH20") (footprint "Package_SO:TSSOP-20_4.4x6.5mm_P0.65mm")
     )
     (path "/00000000-0000-0000-0000-00005f1b616d"
