File: mk4-tlc5940-lpc812/electronics-switching/rev3/rc-light-controller-switching.kicad_sch (KiCad schematic)
At the start: 20 parts, among them J1 Pinheader right-angle 2x17, J2 Pinheader straight 1x06, J3 Pinheader straight 1x06, T1 PMV30UN, T2 PMV30UN, T3 PMV30UN, T4 PMV30UN, T5 PMV30UN, T6 PMV30UN, T7 PMV30UN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

Commit message: Improve file names, BOM and gerbers
Parts:
- U1: value LPC832M101FDH20 -> LPC824M201JDH20
Changed lines of the file:
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@@
     (in_bom yes) (on_board yes)
     (property "Reference" "U1" (id 0) (at 165.1 146.05 0))
-    (property "Value" "LPC832M101FDH20" (id 1) (at 157.48 148.59 0))
+    (property "Value" "LPC824M201JDH20" (id 1) (at 157.48 148.59 0))
     (property "Footprint" "Package_SO:TSSOP-20_4.4x6.5mm_P0.65mm" (id 2) (at 200.66 148.59 0)
       (effects (font (size 1.27 1.27)) hide)
@@
     )
     (path "/00000000-0000-0000-0000-000060f75db2"
-      (reference "U1") (unit 1) (value "LPC832M101FDH20") (footprint "Package_SO:TSSOP-20_4.4x6.5mm_P0.65mm")
+      (reference "U1") (unit 1) (value "LPC824M201JDH20") (footprint "Package_SO:TSSOP-20_4.4x6.5mm_P0.65mm")
     )
     (path "/00000000-0000-0000-0000-000009b5dc2d"
